File: eletronica/aw_201_clock/aw_201_clock.sch (EAGLE design)
At the start: 16 parts, among them IC1 4060N, IC2 4013N, IC3 4026N, IC4 4026N, IC5 4026N, IC6 4026N, IC7 4026N, IC8 4026N, Q1 32.768 Khz

Commit message: 
Parts:
- added C3: 47mF, rcl:C-EU050-024X044
- added D1, D2: 1N4004, diode:1N4004
- added IC9: 4081N, 40xx:4081N
- added LED1: (no value), led:LED5MM
- added R10: 220, resistor:R-EU_0207/10
- added R11, R8: 10M, resistor:R-EU_0207/10
- added R3, R5, R7, R9: 10K, resistor:R-EU_0207/10
- added R4, R6: 1K, resistor:R-EU_0207/10
- added T1, T2, T3: 2N2222, transistor:2N2222
Connections:
- new net N$52: IC9A.I1, R4.1, T1.C
- new net N$53: R3.2, T1.B
- new net N$54: IC9C.O, IC9D.I0
- new net N$55: D1.A, IC3A.RES, IC9A.O
- new net N$56: IC9B.I1, R6.1, T2.C
- new net N$57: R5.2, T2.B
- new net N$58: C3.1, IC2B.R, R7.2
- new net N$59: D1.C, IC6A.CLK
- new net N$60: D2.C, IC8A.CLK
- new net N$61: D2.A, IC5A.RES, IC9B.O
- new net N$62: IC2B.CLK, IC2B.D, IC2B.S, R8.1
- new net N$63: IC7A.RES, IC8A.RES, IC9D.O
- new net N$65: R9.2, T3.B
- new net N$66: LED1.C, R10.2
- new net N$67: R10.1, T3.C
- new net N$68: IC2B.!Q, IC3A.CI, R11.1, R9.1
- net +5V: now also C3.2, IC1P.VDD, IC2P.VDD, IC3P.VDD, IC4P.VDD, IC5P.VDD, IC6P.VDD, IC7P.VDD, IC8P.VDD, IC9P.VDD, LED1.A, R4.2, R6.2
- net GND: now also IC1P.VSS, IC2P.VSS, IC3P.VSS, IC4P.VSS, IC5P.VSS, IC6P.VSS, IC7P.VSS, IC8P.VSS, IC9P.VSS, R11.2, R7.1, R8.2, T1.E, T2.E, T3.E; no longer IC3A.CI, IC3A.RES, IC5A.RES, IC7A.RES, IC8A.RES
- net N$15: now also IC9A.I0
- net N$18: now also R3.1
- net N$28: now also IC9B.I0
- net N$33: now also R5.1
- net N$40: now also IC9C.I0
- net N$41: now also IC9C.I1
- net N$43: now also IC9D.I1
Other:
- moved on the sheet: IC2B, IC4, IC6, Q1, R1

Commit message: 
Parts:
- added D3, D4: 1N4004, diode:1N4004
- added R13, R14: 10K, resistor:R-EU_0207/10
- added S1, S2: PVA2, switch-misc:PVA2
Connections:
- removed net N$59: D1.C, IC6A.CLK
- new net N$64: IC1A.Q13, S12.S, S22.S
- new net N$69: D1.C, D3.A, IC6A.CLK, R14.1, S12.P
- net GND: now also IC2B.CLK, IC2B.D, R13.2, R14.2
- net N$60: now also D4.A, R13.1, S22.P
- net N$62: now also D3.C, D4.C; no longer IC2B.CLK, IC2B.D
Other:
- moved on the sheet: IC1P, IC2P, IC3P, IC4P, IC5P, IC6P, IC7P, IC8P, IC9P
