File: eletronica/aw_601_pongclock/kicad/aw_601_pongclock.sch (KiCad schematic (older format))
At the start: 121 parts

Commit message: 
Parts:
- gave numbers to parts that had none: 121
Connections:
- net Vcc is gone; now on net +5V: U1.24 (Vcc), U6.16 (Vcc), U7.16 (Vcc), U8.16 (Vcc), U9.16 (Vcc)
- net G1: now also D1.17 (C1), U2.18 (O1)
- net G10: now also D1.26 (C10), U3.17 (O2)
- net G11: now also D1.27 (C11), U3.16 (O3)
- net G12: now also D1.28 (C12), U3.15 (O4)
- net G13: now also D1.29 (C13), U3.14 (O5)
- net G14: now also D1.30 (C14), U3.13 (O6)
- net G15: now also D1.31 (C15), U3.12 (O7)
- net G16: now also D1.32 (C16), U3.11 (O8)
- net G17: now also D2.17 (C1), U4.18 (O1)
- net G18: now also D2.18 (C2), U4.17 (O2)
- net G19: now also D2.19 (C3), U4.16 (O3)
- net G2: now also D1.18 (C2), U2.17 (O2)
- net G20: now also D2.20 (C4), U4.15 (O4)
- net G21: now also D2.21 (C5), U4.14 (O5)
- net G22: now also D2.22 (C6), U4.13 (O6)
- net G23: now also D2.23 (C7), U4.12 (O7)
- net G24: now also D2.24 (C8), U4.11 (O8)
- net G25: now also D2.25 (C9), U5.18 (O1)
- net G26: now also D2.26 (C10), U5.17 (O2)
- net G27: now also D2.27 (C11), U5.16 (O3)
- net G28: now also D2.28 (C12), U5.15 (O4)
- net G29: now also D2.29 (C13), U5.14 (O5)
- net G3: now also D1.19 (C3), U2.16 (O3)
- net G30: now also D2.30 (C14), U5.13 (O6)
- net G31: now also D2.31 (C15), U5.12 (O7)
- net G32: now also D2.32 (C16), U5.11 (O8)
- net G4: now also D1.20 (C4), U2.15 (O4)
- net G5: now also D1.21 (C5), U2.14 (O5)
- net G6: now also D1.22 (C6), U2.13 (O6)
- net G7: now also D1.23 (C7), U2.12 (O7)
- net G8: now also D1.24 (C8), U2.11 (O8)
- net G9: now also D1.25 (C9), U3.18 (O1)
- net GND: now also U1.23 (INHIBIT)
- net V1: now also Q1.2 (E), R11.1
- net V10: now also Q10.2 (E), R20.1
- net V11: now also Q11.2 (E), R21.1
- net V12: now also Q12.2 (E), R22.1
- net V13: now also Q13.2 (E), R23.1
- net V14: now also Q14.2 (E), R24.1
- net V15: now also Q15.2 (E), R25.1
- net V16: now also Q16.2 (E), R26.1
- net V17: now also Q17.2 (E), R36.1
- net V18: now also Q18.2 (E), R37.1
- net V19: now also Q19.2 (E), R38.1
- net V2: now also Q2.2 (E), R12.1
- net V20: now also Q20.2 (E), R39.1
- net V21: now also Q21.2 (E), R40.1
- net V22: now also Q22.2 (E), R41.1
- net V23: now also Q23.2 (E), R42.1
- net V24: now also Q24.2 (E), R43.1
- net V25: now also Q25.2 (E), R44.1
- net V26: now also Q26.2 (E), R45.1
- net V27: now also Q27.2 (E), R46.1
- net V28: now also Q28.2 (E), R47.1
- net V29: now also Q29.2 (E), R48.1
- net V3: now also Q3.2 (E), R13.1
- net V30: now also Q30.2 (E), R49.1
- net V31: now also Q31.2 (E), R50.1
- net V32: now also Q32.2 (E), R51.1
- net V4: now also Q4.2 (E), R14.1
- net V5: now also Q5.2 (E), R15.1
- net V6: now also Q6.2 (E), R16.1
- net V7: now also Q7.2 (E), R17.1
- net V8: now also Q8.2 (E), R18.1
- net V9: now also Q9.2 (E), R19.1
- net at IC1.2 ((RXD)PD0): now also U1.2 (D1); no longer U1.22 (D4)
- net at IC1.26 ((ADC3)PC3), SW1.2, SW2.2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: now also SW3.2
- net at IC1.3 ((TXD)PD1): now also U1.3 (D2)
- net at IC1.4 ((INT0)PD2): now also U1.21 (D3)
- net at IC1.5 ((INT1)PD3): now also U1.22 (D4); no longer U1.1 (STROBE)
- net at IC1.6 ((XCK/T0)PD4): now also U1.1 (STROBE)
- net at U8.11 (QP7): now also R43.2
- net at U8.12 (QP6): now also R42.2
- net at U8.13 (QP5): now also R41.2
- net at U8.14 (QP4): now also R40.2
- net at U8.4 (QP0): now also R36.2
- net at U8.5 (QP1): now also R37.2
- net at U8.6 (QP2): now also R38.2
- net at U8.7 (QP3): now also R39.2
- net at U9.11 (QP7): now also R51.2
- net at U9.12 (QP6): now also R50.2
- net at U9.13 (QP5): now also R49.2
- net at U9.14 (QP4): now also R48.2
- net at U9.4 (QP0): now also R44.2
- net at U9.5 (QP1): now also R45.2
- net at U9.6 (QP2): now also R46.2
- net at U9.7 (QP3): now also R47.2
- net at U1.10 (S2): now also U2.3 (I3), U3.3 (I3)
- net at U1.11 (S0): now also U2.1 (I1), U3.1 (I1)
- net at U4.3 (I3), U5.3 (I3): now also U1.20 (S10); no longer U1.13 (S13)
- net at U4.2 (I2), U5.2 (I2): now also U1.17 (S9); no longer U1.14 (S12)
- net at U4.5 (I5), U5.5 (I5): now also U1.14 (S12); no longer U1.15 (S15)
- net at U4.4 (I4), U5.4 (I4): now also U1.19 (S11); no longer U1.16 (S14)
- net at U2.7 (I7), U3.7 (I7): now also U1.5 (S6); no longer U1.17 (S9)
- net at U2.6 (I6), U3.6 (I6): now also U1.6 (S5); no longer U1.18 (S8)
- net at U4.1 (I1), U5.1 (I1): now also U1.18 (S8); no longer U1.19 (S11)
- net at U2.8 (I8), U3.8 (I8): now also U1.4 (S7); no longer U1.20 (S10)
- net at U2.5 (I5), U3.5 (I5): now also U1.7 (S4); no longer U1.4 (S7)
- net at U2.4 (I4), U3.4 (I4): now also U1.8 (S3); no longer U1.5 (S6)
- net at U2.2 (I2), U3.2 (I2): now also U1.9 (S1); no longer U1.7 (S4)
- net at U4.6 (I6), U5.6 (I6): now also U1.13 (S13)
- net at U4.7 (I7), U5.7 (I7): now also U1.16 (S14)
- net at U4.8 (I8), U5.8 (I8): now also U1.15 (S15)
- no-connect marks 10 -> 14
Other:
- moved on the sheet: R11, R12, R13, R14, R15, R16, R17, R18, R36, R37, R38, R39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
