File: eletronica/2_inprogress/aw_601_pongclock/kicad/aw_601_pongclock.sch (KiCad schematic (older format))
At the start: 121 parts, among them IC1 ATMEGA8-P, Q1 2N3904G, Q10 2N3904G, Q11 2N3904G, Q12 2N3904G, Q13 2N3904G, Q14 2N3904G, Q15 2N3904G, Q16 2N3904G, Q17 2N3904G, Q18 2N3904G, Q19 2N3904G, Q2 2N3904G, Q20 2N3904G, Q21 2N3904G, Q22 2N3904G, Q23 2N3904G, Q24 2N3904G, Q25 2N3904G, Q26 2N3904G, Q27 2N3904G, Q28 2N3904G, Q29 2N3904G, Q3 2N3904G, Q30 2N3904G, Q31 2N3904G, Q32 2N3904G, Q4 2N3904G, Q5 2N3904G, Q6 2N3904G, Q7 2N3904G, Q8 2N3904G, Q9 2N3904G, SW1 SW_PUSH, SW2 SW_PUSH, SW3 SW_PUSH, SW4 SW_PUSH, U1 4514, U2 ULN2803, U3 ULN2803, U4 ULN2803, U5 ULN2803, U6 74HC4094, U7 74HC4094, U8 74HC4094, U9 74HC4094, X1 16Mhz

Commit message: 
Parts:
- removed R11, R12, R13, R14, R15, R16, R17, R18, R19, R20, R21, R22, R23, R24, R25, R26, R36, R37, R38, R39, R40, R41, R42, R43, R44, R45, R46, R47, R48, R49, R50, R51: 10K, ~, symbol R
Connections:
- net V1: now also U6.4 (QP0)
- net V10: now also U7.5 (QP1)
- net V11: now also U7.6 (QP2)
- net V12: now also U7.7 (QP3)
- net V13: now also U7.14 (QP4)
- net V14: now also U7.13 (QP5)
- net V15: now also U7.12 (QP6)
- net V16: now also U7.11 (QP7)
- net V17: now also U8.4 (QP0)
- net V18: now also U8.5 (QP1)
- net V19: now also U8.6 (QP2)
- net V2: now also U6.5 (QP1)
- net V20: now also U8.7 (QP3)
- net V21: now also U8.14 (QP4)
- net V22: now also U8.13 (QP5)
- net V23: now also U8.12 (QP6)
- net V24: now also U8.11 (QP7)
- net V25: now also U9.4 (QP0)
- net V26: now also U9.5 (QP1)
- net V27: now also U9.6 (QP2)
- net V28: now also U9.7 (QP3)
- net V29: now also U9.14 (QP4)
- net V3: now also U6.6 (QP2)
- net V30: now also U9.13 (QP5)
- net V31: now also U9.12 (QP6)
- net V32: now also U9.11 (QP7)
- net V4: now also U6.7 (QP3)
- net V5: now also U6.14 (QP4)
- net V6: now also U6.13 (QP5)
- net V7: now also U6.12 (QP6)
- net V8: now also U6.11 (QP7)
- net V9: now also U7.4 (QP0)
- net OE: now reaches IC1.11 ((T1)PD5), U6.15 (OE), U7.15 (OE), U8.15 (OE), U9.15 (OE)
- net DATA0: now reaches IC1.14 ((ICP)PB0), U6.2 (D)
- net DATA1: now reaches IC1.15 ((OC1A)PB1), U7.2 (D)
- net DATA2: now reaches IC1.16 ((~SS~/OC1B)PB2), U8.2 (D)
- net DATA3: now reaches IC1.17 ((MOSI/OC2)PB3), U9.2 (D)
- net CP: now reaches IC1.18 ((MISO)PB4), U6.3 (CP), U7.3 (CP), U8.3 (CP), U9.3 (CP)
- net STR: now reaches IC1.19 ((SCK)PB5), U6.1 (STR), U7.1 (STR), U8.1 (STR), U9.1 (STR)
- net D1: now reaches IC1.2 ((RXD)PD0), U1.2 (D1)
- net D2: now reaches IC1.3 ((TXD)PD1), U1.3 (D2)
- net D3: now reaches IC1.4 ((INT0)PD2), U1.21 (D3)
- net D4: now reaches IC1.5 ((INT1)PD3), U1.22 (D4)
- net STRB: now reaches IC1.6 ((XCK/T0)PD4), U1.1 (STROBE)

Commit message: 
Parts:
- U1: footprint ~ -> DIP-24__600
- U2, U3, U4, U5, U6, U7, U8, U9: footprint ~ -> DIP-16_300
Changed lines of the file:
@@
-EESchema Schematic File Version 2  date 12/06/2013 17:21:00
+EESchema Schematic File Version 2  date 13/06/2013 09:16:40
 LIBS:power
 LIBS:device
@@
 LIBS:contrib
 LIBS:valves
+LIBS:kicad
 LIBS:aw_601_pongclock-cache
 EELAYER 27 0
@@
 Sheet 1 1
 Title "AW601 Pong Clock"
-Date "12 jun 2013"
+Date "13 jun 2013"
 Rev ""
 Comp "Imperial Electronics"
@@
 F 0 "U7" H 7900 4700 60  0000 C CNN
 F 1 "74HC4094" H 7750 3500 60  0000 C CNN
-F 2 "~" H 7500 4100 60  0000 C CNN
+F 2 "DIP-16_300" H 7500 4100 60  0000 C CNN
 F 3 "~" H 7500 4100 60  0000 C CNN
 	1    7500 4100
@@
 F 0 "U8" H 10950 2600 60  0000 C CNN
 F 1 "74HC4094" H 10800 1400 60  0000 C CNN
-F 2 "~" H 10550 2000 60  0000 C CNN
+F 2 "DIP-16_300" H 10550 2000 60  0000 C CNN
 F 3 "~" H 10550 2000 60  0000 C CNN
 	1    10550 2000
@@
 F 0 "U9" H 10950 4700 60  0000 C CNN
 F 1 "74HC4094" H 10800 3500 60  0000 C CNN
-F 2 "~" H 10550 4100 60  0000 C CNN
+F 2 "DIP-16_300" H 10550 4100 60  0000 C CNN
 F 3 "~" H 10550 4100 60  0000 C CNN
 	1    10550 4100
@@
 F 0 "U1" H 2600 6750 60  0000 C CNN
 F 1 "4514" H 2600 4950 60  0000 C CNN
-F 2 "~" H 2300 5900 60  0000 C CNN
+F 2 "DIP-24__600" H 2300 5900 60  0000 C CNN
 F 3 "~" H 2300 5900 60  0000 C CNN
 	1    2300 5900
@@
 F 0 "U2" H 4800 6150 60  0000 C CNN
 F 1 "ULN2803" H 4650 5000 60  0000 C CNN
-F 2 "~" H 4500 5600 60  0000 C CNN
+F 2 "DIP-16_300" H 4500 5600 60  0000 C CNN
 F 3 "~" H 4500 5600 60  0000 C CNN
 	1    4500 5600
@@
 F 0 "U3" H 4800 7450 60  0000 C CNN
 F 1 "ULN2803" H 4650 6300 60  0000 C CNN
-F 2 "~" H 4500 6900 60  0000 C CNN
+F 2 "DIP-16_300" H 4500 6900 60  0000 C CNN
 F 3 "~" H 4500 6900 60  0000 C CNN
 	1    4500 6900
@@
 F 0 "U4" H 4800 8750 60  0000 C CNN
 F 1 "ULN2803" H 4650 7600 60  0000 C CNN
-F 2 "~" H 4500 8200 60  0000 C CNN
+F 2 "DIP-16_300" H 4500 8200 60  0000 C CNN
 F 3 "~" H 4500 8200 60  0000 C CNN
 	1    4500 8200
@@
 F 0 "U5" H 4800 10050 60  0000 C CNN
 F 1 "ULN2803" H 4650 8900 60  0000 C CNN
-F 2 "~" H 4500 9500 60  0000 C CNN
+F 2 "DIP-16_300" H 4500 9500 60  0000 C CNN
 F 3 "~" H 4500 9500 60  0000 C CNN
 	1    4500 9500
@@
 F 0 "U6" H 7850 2600 60  0000 C CNN
 F 1 "74HC4094" H 7700 1400 60  0000 C CNN
-F 2 "~" H 7450 2000 60  0000 C CNN
+F 2 "DIP-16_300" H 7450 2000 60  0000 C CNN
 F 3 "~" H 7450 2000 60  0000 C CNN
 	1    7450 2000
