File: eletronica/2_inprogress/aw_601_pongclock/kicad/aw_601_pongclock.kicad_pcb (KiCad board)
At the start: 2 copper layers, 94 parts, among them CON1 BARREL_JACK, IC1 ATMEGA8-P, Q1 2N3904G, Q10 2N3904G, Q11 2N3904G, Q12 2N3904G, Q13 2N3904G, Q14 2N3904G, Q15 2N3904G, Q16 2N3904G, Q17 2N3904G, Q18 2N3904G, Q19 2N3904G, Q2 2N3904G, Q20 2N3904G, Q21 2N3904G, Q22 2N3904G, Q23 2N3904G, Q24 2N3904G, Q25 2N3904G, Q26 2N3904G, Q27 2N3904G, Q28 2N3904G, Q29 2N3904G, Q3 2N3904G, Q30 2N3904G, Q31 2N3904G, Q32 2N3904G, Q4 2N3904G, Q5 2N3904G, Q6 2N3904G, Q7 2N3904G, Q8 2N3904G, Q9 2N3904G, SW1 SW_PUSH, SW2 SW_PUSH, SW3 SW_PUSH, SW4 SW_PUSH, U1 4514, U10 DS1307, U2 ULN2803, U3 ULN2803, U4 ULN2803, U5 ULN2803, U6 74HC4094, U7 74HC4094, U8 74HC4094, U9 74HC4094, X1 16Mhz, X2 32kHz

Commit message: 
Connections:
- Q1 pad 1: (no net) -> N-000001
- Q10 pad 1: (no net) -> N-000009
- Q11 pad 1: (no net) -> N-0000010
- Q12 pad 1: (no net) -> N-000007
- Q13 pad 1: (no net) -> N-0000011
- Q14 pad 1: (no net) -> N-0000012
- Q15 pad 1: (no net) -> N-0000022
- Q16 pad 1: (no net) -> N-0000049
- Q17 pad 1: (no net) -> N-0000050
- Q18 pad 1: (no net) -> N-0000054
- Q19 pad 1: (no net) -> N-0000053
- Q2 pad 1: (no net) -> N-0000014
- Q20 pad 1: (no net) -> N-0000052
- Q21 pad 1: (no net) -> N-0000044
- Q22 pad 1: (no net) -> N-0000051
- Q23 pad 1: (no net) -> N-0000045
- Q24 pad 1: (no net) -> N-0000043
- Q25 pad 1: (no net) -> N-0000046
- Q26 pad 1: (no net) -> N-0000047
- Q27 pad 1: (no net) -> N-0000048
- Q28 pad 1: (no net) -> N-0000059
- Q28 pad 2: N-0000058 -> /V28
- Q29 pad 1: (no net) -> N-0000060
- Q29 pad 2: N-0000059 -> /V29
- Q3 pad 1: (no net) -> N-0000013
- Q30 pad 1: (no net) -> N-0000058
- Q30 pad 2: N-0000057 (its old number) -> /V30
- Q31 pad 1: (no net) -> N-0000061
- Q31 pad 2: N-0000060 -> /V31
- Q32 pad 1: (no net) -> N-0000062
- Q4 pad 1: (no net) -> N-000004
- Q5 pad 1: (no net) -> N-000003
- Q6 pad 1: (no net) -> N-000002
- Q7 pad 1: (no net) -> N-0000015
- Q8 pad 1: (no net) -> N-0000016
- Q9 pad 1: (no net) -> N-000008
- R10 pad 1: (no net) -> N-0000015
- R27 pad 1: (no net) -> N-0000016
- R28 pad 1: (no net) -> N-000008
- R29 pad 1: (no net) -> N-000009
- R30 pad 1: (no net) -> N-0000010
- R31 pad 1: (no net) -> N-000007
- R32 pad 1: (no net) -> N-0000011
- R33 pad 1: (no net) -> N-0000012
- R34 pad 1: (no net) -> N-0000022
- R35 pad 1: (no net) -> N-0000049
- R4 pad 1: (no net) -> N-000001
- R5 pad 1: (no net) -> N-0000014
- R52 pad 1: (no net) -> N-0000050
- R53 pad 1: (no net) -> N-0000054
- R54 pad 1: (no net) -> N-0000053
- R55 pad 1: (no net) -> N-0000052
- R56 pad 1: (no net) -> N-0000044
- R57 pad 1: (no net) -> N-0000051
- R58 pad 1: (no net) -> N-0000045
- R59 pad 1: (no net) -> N-0000043
- R6 pad 1: (no net) -> N-0000013
- R60 pad 1: (no net) -> N-0000046
- R61 pad 1: (no net) -> N-0000047
- R62 pad 1: (no net) -> N-0000048
- R63 pad 1: N-0000058 -> N-0000059
- R64 pad 1: N-0000059 -> N-0000060
- R65 pad 1: N-0000057 (its old number) -> N-0000058
- R66 pad 1: N-0000060 -> N-0000061
- R67 pad 1: (no net) -> N-0000062
- R7 pad 1: (no net) -> N-000004
- R8 pad 1: (no net) -> N-000003
- R9 pad 1: (no net) -> N-000002
- U9 pad 12: (no net) -> /V31
- U9 pad 13: (no net) -> /V30
- U9 pad 14: (no net) -> /V29
- U9 pad 7: (no net) -> /V28
Routing:
- net (no net): track 934.4 -> 0.00 mm
- net N-0000044: track 0.00 -> 60.3 mm
- net N-0000011: track 0.00 -> 55.2 mm
- net N-0000057 (its old number): track 54.5 -> 0.00 mm
- net N-000003: track 0.00 -> 54.3 mm
- net N-0000059: track 71.5 -> 18.8 mm
- net N-0000051: track 0.00 -> 47.1 mm
- net N-000001: track 0.00 -> 43.8 mm
- net N-000008: track 0.00 -> 42.5 mm
- net N-0000012: track 0.00 -> 42.0 mm
- net N-000002: track 0.00 -> 41.8 mm
- net N-0000014: track 0.00 -> 38.2 mm
- net N-0000050: track 0.00 -> 37.4 mm
- net N-0000046: track 0.00 -> 37.4 mm
- net N-000009: track 0.00 -> 36.9 mm
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- added copper zone on B.Cu, net GND
- added copper zone on F.Cu, net GND

Commit message: 
Parts:
- moved U2 2.54 mm to (58.4, 158.8)
- moved U5 2.54 mm to (154.9, 158.8)
- moved D2 1.27 mm to (137.2, 119.4)
- moved D1 1.27 mm to (73.7, 119.4)
Routing:
- net +5V: track 973.6 -> 970.8 mm
- net N-0000039: track 73.2 -> 70.7 mm
- net N-0000055: track 100.1 -> 97.6 mm
- net N-0000040: track 82.3 -> 79.8 mm
- net N-0000027: track 90.0 -> 87.4 mm
- net N-0000026: track 60.5 -> 58.0 mm
- net N-0000023: track 65.1 -> 62.5 mm
- net N-0000057: track 91.2 -> 88.7 mm
- net N-0000056: track 98.4 -> 95.9 mm
- net N-0000042: track 83.6 -> 81.1 mm
- net N-0000041: track 88.5 -> 85.9 mm
- net N-0000037: track 77.0 -> 74.5 mm
- net N-0000029: track 112.6 -> 110.1 mm
- net N-0000028: track 110.1 -> 107.5 mm
- net N-0000025: track 69.6 -> 67.1 mm
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Other:
- board text added: "AW 2013"
- board text added: "SUPER PONG CLOCK"
