File: eletronica/3_done/aw_301_runner/aw_301_runner.sch (EAGLE design)
At the start: 6 parts, among them IC1 ATTINY2313V

Commit message: 
Parts:
- added Q1: (no value), special:XTAL
Connections:
- new net N$13: IC1.XTAL1, Q1.1
- new net N$6: IC1.XTAL2, Q1.2
Other:
- moved on the sheet: C1
Changed lines of the file:
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@@
 <part name="GND4" library="supply1" deviceset="GND" device=""/>
 <part name="C2" library="resistor" deviceset="CPOL-EU" device="E2.5-6" value="100mF"/>
+<part name="Q1" library="special" deviceset="XTAL" device=""/>
 </parts>
 <sheets>
@@
 <attribute name="VALUE" x="99.06" y="81.28" size="1.778" layer="96"/>
 </instance>
-<instance part="C1" gate="G$1" x="71.12" y="30.48"/>
+<instance part="C1" gate="G$1" x="60.96" y="30.48"/>
 <instance part="GND2" gate="1" x="104.14" y="71.12"/>
-<instance part="GND3" gate="1" x="71.12" y="12.7"/>
+<instance part="GND3" gate="1" x="60.96" y="12.7"/>
 <instance part="SG1" gate="G$1" x="129.54" y="22.86" rot="R270"/>
 <instance part="GND4" gate="1" x="142.24" y="71.12"/>
 <instance part="C2" gate="G$1" x="116.84" y="22.86" rot="R90"/>
+<instance part="Q1" gate="G$1" x="68.58" y="40.64" rot="R90"/>
 </instances>
 <busses>
@@
 <pinref part="C1" gate="G$1" pin="-"/>
 <pinref part="GND3" gate="1" pin="GND"/>
-<wire x1="71.12" y1="15.24" x2="71.12" y2="22.86" width="0.1524" layer="91"/>
+<wire x1="60.96" y1="15.24" x2="60.96" y2="22.86" width="0.1524" layer="91"/>
 <pinref part="IC1" gate="G$1" pin="GND"/>
-<wire x1="71.12" y1="22.86" x2="71.12" y2="25.4" width="0.1524" layer="91"/>
+<wire x1="60.96" y1="22.86" x2="60.96" y2="25.4" width="0.1524" layer="91"/>
 <wire x1="76.2" y1="30.48" x2="76.2" y2="22.86" width="0.1524" layer="91"/>
-<wire x1="76.2" y1="22.86" x2="71.12" y2="22.86" width="0.1524" layer="91"/>
-<junction x="71.12" y="22.86"/>
+<wire x1="76.2" y1="22.86" x2="60.96" y2="22.86" width="0.1524" layer="91"/>
+<junction x="60.96" y="22.86"/>
 </segment>
 <segment>
@@
 <segment>
 <pinref part="SW1" gate="A" pin="9"/>
-<wire x1="116.84" y1="58.42" x2="71.12" y2="58.42" width="0.1524" layer="91"/>
+<wire x1="116.84" y1="58.42" x2="60.96" y2="58.42" width="0.1524" layer="91"/>
 <pinref part="IC1" gate="G$1" pin="VCC"/>
 <pinref part="C1" gate="G$1" pin="+"/>
-<wire x1="71.12" y1="33.02" x2="76.2" y2="33.02" width="0.1524" layer="91"/>
-<junction x="71.12" y="33.02"/>
-<wire x1="71.12" y1="58.42" x2="71.12" y2="33.02" width="0.1524" layer="91"/>
+<wire x1="60.96" y1="33.02" x2="76.2" y2="33.02" width="0.1524" layer="91"/>
+<junction x="60.96" y="33.02"/>
+<wire x1="60.96" y1="58.42" x2="60.96" y2="33.02" width="0.1524" layer="91"/>
 </segment>
 </net>
@@
 </segment>
 </net>
+<net name="N$6" class="0">
+<segment>
+<pinref part="Q1" gate="G$1" pin="2"/>
+<pinref part="IC1" gate="G$1" pin="XTAL2"/>
+<wire x1="68.58" y1="45.72" x2="76.2" y2="45.72" width="0.1524" layer="91"/>
+<wire x1="76.2" y1="45.72" x2="76.2" y2="43.18" width="0.1524" layer="91"/>
+</segment>
+</net>
+<net name="N$13" class="0">
+<segment>
+<pinref part="IC1" gate="G$1" pin="XTAL1"/>
+<wire x1="76.2" y1="38.1" x2="76.2" y2="35.56" width="0.1524" layer="91"/>
+<pinref part="Q1" gate="G$1" pin="1"/>
+<wire x1="76.2" y1="35.56" x2="68.58" y2="35.56" width="0.1524" layer="91"/>
+</segment>
+</net>
