File: eletronica/4_other/apunk/apunk.sch (KiCad schematic (older format))
At the start: 11 parts, among them J1 JACK_2P, U1 LM556N

Commit message: 
Parts:
- removed U1: LM556N, symbol LM556N
- added U? (x2): LM555N, symbol LM555N
Connections:
- wire segments 29 -> 33
Other:
- moved on the sheet: C1, C2, C3, J1, R2, R3, RV2
Changed lines of the file:
@@
 Sheet 1 1
 Title ""
-Date "28 jun 2013"
+Date "29 jun 2013"
 Rev ""
 Comp ""
@@
 L POT RV2
 U 1 1 51CDBDF3
-P 4500 3550
-F 0 "RV2" H 4500 3450 50  0000 C CNN
-F 1 "470K" H 4500 3550 50  0000 C CNN
-F 2 "~" H 4500 3550 60  0000 C CNN
-F 3 "~" H 4500 3550 60  0000 C CNN
-	1    4500 3550
+P 4500 3750
+F 0 "RV2" H 4500 3650 50  0000 C CNN
+F 1 "470K" H 4500 3750 50  0000 C CNN
+F 2 "~" H 4500 3750 60  0000 C CNN
+F 3 "~" H 4500 3750 60  0000 C CNN
+	1    4500 3750
 	0    1    1    0
 $EndComp
@@
 	0    -1   -1   0
 $EndComp
-$Comp
-L LM556N U1
-U 1 1 51CDC29B
-P 2800 2900
-F 0 "U1" H 2800 3000 70  0000 C CNN
-F 1 "LM556N" H 2800 2800 70  0000 C CNN
-F 2 "" H 2800 2900 60  0000 C CNN
-F 3 "" H 2800 2900 60  0000 C CNN
-	1    2800 2900
-	1    0    0    -1
-$EndComp
-Wire Wire Line
-	4500 3300 4650 3300
+Wire Wire Line
+	4500 3500 4650 3500
 Wire Wire Line
 	4050 2350 4050 2100
 Connection ~ 4200 2100
 Wire Wire Line
-	4650 3300 4650 3550
-Connection ~ 4500 3300
+	4650 3500 4650 3750
+Connection ~ 4500 3500
 Wire Wire Line
 	4200 2600 3500 2600
-Wire Wire Line
-	3500 3450 4100 3450
 $Comp
 L R R1
@@
 	3700 2800 3500 2800
 Wire Wire Line
-	3700 1900 3700 3800
+	3700 1900 3700 2800
+Wire Wire Line
+	3700 2800 3700 4000
 Wire Wire Line
 	3700 1900 2100 1900
 Wire Wire Line
-	2100 1900 2100 2300
+	2100 1900 2100 2400
 Connection ~ 3700 2800
 $Comp
 L C C1
 U 1 1 51CDC33B
-P 3700 4000
-F 0 "C1" H 3700 4100 40  0000 L CNN
-F 1 "10n" H 3706 3915 40  0000 L CNN
-F 2 "~" H 3738 3850 30  0000 C CNN
-F 3 "~" H 3700 4000 60  0000 C CNN
-	1    3700 4000
+P 3700 4200
+F 0 "C1" H 3700 4300 40  0000 L CNN
+F 1 "10n" H 3706 4115 40  0000 L CNN
+F 2 "~" H 3738 4050 30  0000 C CNN
+F 3 "~" H 3700 4200 60  0000 C CNN
+	1    3700 4200
 	1    0    0    -1
 $EndComp
@@
 L GND #PWR02
 U 1 1 51CDC35E
-P 4500 4300
-F 0 "#PWR02" H 4500 4300 30  0001 C CNN
-F 1 "GND" H 4500 4230 30  0001 C CNN
-F 2 "" H 4500 4300 60  0000 C CNN
-F 3 "" H 4500 4300 60  0000 C CNN
-	1    4500 4300
+P 4500 4500
+F 0 "#PWR02" H 4500 4500 30  0001 C CNN
+F 1 "GND" H 4500 4430 30  0001 C CNN
+F 2 "" H 4500 4500 60  0000 C CNN
+F 3 "" H 4500 4500 60  0000 C CNN
+	1    4500 4500
 	1    0    0    -1
 $EndComp
@@
 	3500 2000 1850 2000
 Wire Wire Line
-	1850 2000 1850 3050
-Wire Wire Line
-	1850 3050 2100 3050
+	1850 2000 1850 3250
+Wire Wire Line
+	1850 3250 2100 3250
 $Comp
 L +9V #PWR03
 U 1 1 51CDC3CB
-P 2100 2800
-F 0 "#PWR03" H 2100 2770 20  0001 C CNN
-F 1 "+9V" H 2100 2910 30  0000 C CNN
-F 2 "" H 2100 2800 60  0000 C CNN
-F 3 "" H 2100 2800 60  0000 C CNN
-	1    2100 2800
-	1    0    0    -1
-$EndComp
-NoConn ~ 2100 2550
-NoConn ~ 2100 3300
+P 2100 2900
+F 0 "#PWR03" H 2100 2870 20  0001 C CNN
+F 1 "+9V" H 2100 3010 30  0000 C CNN
+F 2 "" H 2100 2900 60  0000 C CNN
+F 3 "" H 2100 2900 60  0000 C CNN
+	1    2100 2900
+	1    0    0    -1
+$EndComp
+NoConn ~ 2100 2650
+NoConn ~ 2100 3500
 $Comp
 L +9V #PWR04
 U 1 1 51CDC3DB
-P 2100 3550
-F 0 "#PWR04" H 2100 3520 20  0001 C CNN
-F 1 "+9V" H 2100 3660 30  0000 C CNN
-F 2 "" H 2100 3550 60  0000 C CNN
-F 3 "" H 2100 3550 60  0000 C CNN
-	1    2100 3550
-	1    0    0    -1
-$EndComp
-Wire Wire Line
-	3500 3250 4100 3250
+P 2100 3750
+F 0 "#PWR04" H 2100 3720 20  0001 C CNN
+F 1 "+9V" H 2100 3860 30  0000 C CNN
+F 2 "" H 2100 3750 60  0000 C CNN
+F 3 "" H 2100 3750 60  0000 C CNN
+	1    2100 3750
+	1    0    0    -1
+$EndComp
 $Comp
 L CP1 C3
 U 1 1 51CDC41A
-P 5100 3050
-F 0 "C3" H 5150 3150 50  0000 L CNN
-F 1 "10u" H 5150 2950 50  0000 L CNN
-F 2 "~" H 5100 3050 60  0000 C CNN
-F 3 "~" H 5100 3050 60  0000 C CNN
-	1    5100 3050
+P 5100 3250
+F 0 "C3" H 5150 3350 50  0000 L CNN
+F 1 "10u" H 5150 3150 50  0000 L CNN
+F 2 "~" H 5100 3250 60  0000 C CNN
+F 3 "~" H 5100 3250 60  0000 C CNN
+	1    5100 3250
 	0    -1   -1   0
 $EndComp
@@
 L R R3
 U 1 1 51CDC427
-P 5800 3300
-F 0 "R3" V 5880 3300 40  0000 C CNN
-F 1 "4K7" V 5807 3301 40  0000 C CNN
-F 2 "~" V 5730 3300 30  0000 C CNN
-F 3 "~" H 5800 3300 30  0000 C CNN
-	1    5800 3300
+P 5800 3500
+F 0 "R3" V 5880 3500 40  0000 C CNN
+F 1 "4K7" V 5807 3501 40  0000 C CNN
+F 2 "~" V 5730 3500 30  0000 C CNN
+F 3 "~" H 5800 3500 30  0000 C CNN
+	1    5800 3500
 	-1   0    0    1
 $EndComp
@@
 L R R2
 U 1 1 51CDC43C
-P 5550 3050
-F 0 "R2" V 5630 3050 40  0000 C CNN
-F 1 "10K" V 5557 3051 40  0000 C CNN
-F 2 "~" V 5480 3050 30  0000 C CNN
-F 3 "~" H 5550 3050 30  0000 C CNN
-	1    5550 3050
+P 5550 3250
+F 0 "R2" V 5630 3250 40  0000 C CNN
+F 1 "10K" V 5557 3251 40  0000 C CNN
+F 2 "~" V 5480 3250 30  0000 C CNN
+F 3 "~" H 5550 3250 30  0000 C CNN
+	1    5550 3250
 	0    1    1    0
 $EndComp
 Wire Wire Line
-	4900 3050 3500 3050
-Wire Wire Line
-	4100 3800 4500 3800
-Wire Wire Line
-	4100 3250 4100 3800
-Connection ~ 4100 3450
+	4900 3250 3500 3250
+Wire Wire Line
+	4100 4000 4500 4000
 $Comp
 L C C2
 U 1 1 51CDC505
-P 4500 4000
-F 0 "C2" H 4500 4100 40  0000 L CNN
-F 1 "100n" H 4506 3915 40  0000 L CNN
-F 2 "~" H 4538 3850 30  0000 C CNN
-F 3 "~" H 4500 4000 60  0000 C CNN
-	1    4500 4000
-	1    0    0    -1
-$EndComp
-Wire Wire Line
-	4500 4200 3700 4200
+P 4500 4200
+F 0 "C2" H 4500 4300 40  0000 L CNN
+F 1 "100n" H 4506 4115 40  0000 L CNN
+F 2 "~" H 4538 4050 30  0000 C CNN
+F 3 "~" H 4500 4200 60  0000 C CNN
+	1    4500 4200
+	1    0    0    -1
+$EndComp
+Wire Wire Line
+	4500 4400 3700 4400
 $Comp
 L +9V #PWR05
 U 1 1 51CDC55B
-P 4500 3250
-F 0 "#PWR05" H 4500 3220 20  0001 C CNN
-F 1 "+9V" H 4500 3360 30  0000 C CNN
-F 2 "" H 4500 3250 60  0000 C CNN
-F 3 "" H 4500 3250 60  0000 C CNN
-	1    4500 3250
-	1    0    0    -1
-$EndComp
-Wire Wire Line
-	4500 3300 4500 3250
+P 4500 3450
+F 0 "#PWR05" H 4500 3420 20  0001 C CNN
+F 1 "+9V" H 4500 3560 30  0000 C CNN
+F 2 "" H 4500 3450 60  0000 C CNN
+F 3 "" H 4500 3450 60  0000 C CNN
+	1    4500 3450
+	1    0    0    -1
+$EndComp
+Wire Wire Line
+	4500 3500 4500 3450
 Wire Wire Line
 	4200 2100 4200 2000
@@
 L GND #PWR06
 U 1 1 51CDC6D7
-P 5800 3600
-F 0 "#PWR06" H 5800 3600 30  0001 C CNN
-F 1 "GND" H 5800 3530 30  0001 C CNN
-F 2 "" H 5800 3600 60  0000 C CNN
-F 3 "" H 5800 3600 60  0000 C CNN
-	1    5800 3600
-	1    0    0    -1
-$EndComp
-Wire Wire Line
-	5800 3550 5800 3600
+P 5800 3800
+F 0 "#PWR06" H 5800 3800 30  0001 C CNN
+F 1 "GND" H 5800 3730 30  0001 C CNN
+F 2 "" H 5800 3800 60  0000 C CNN
+F 3 "" H 5800 3800 60  0000 C CNN
+	1    5800 3800
+	1    0    0    -1
+$EndComp
+Wire Wire Line
+	5800 3750 5800 3800
 $Comp
 L JACK_2P J1
 U 1 1 51CDC71A
-P 6550 2900
-F 0 "J1" H 6200 2700 60  0000 C CNN
-F 1 "JACK_2P" H 6400 3150 60  0000 C CNN
-F 2 "~" H 6550 2900 60  0000 C CNN
-F 3 "~" H 6550 2900 60  0000 C CNN
-	1    6550 2900
+P 6550 3100
+F 0 "J1" H 6200 2900 60  0000 C CNN
+F 1 "JACK_2P" H 6400 3350 60  0000 C CNN
+F 2 "~" H 6550 3100 60  0000 C CNN
+F 3 "~" H 6550 3100 60  0000 C CNN
+	1    6550 3100
 	-1   0    0    1
 $EndComp
 Wire Wire Line
-	5800 3550 5950 3550
-Wire Wire Line
-	5950 3550 5950 2800
-Wire Wire Line
-	5950 2800 6100 2800
-Wire Wire Line
-	6100 2900 5950 2900
-Connection ~ 5950 2900
-Wire Wire Line
-	5800 3050 6100 3050
-Wire Wire Line
-	4500 4200 4500 4300
+	5950 3750 5800 3750
+Wire Wire Line
+	5950 3000 5950 3100
+Wire Wire Line
+	5950 3100 5950 3750
+Wire Wire Line
+	5950 3000 6100 3000
+Wire Wire Line
+	6100 3100 5950 3100
+Connection ~ 5950 3100
+Wire Wire Line
+	5800 3250 6100 3250
+Wire Wire Line
+	4500 4400 4500 4500
 $Comp
 L BATTERY BT1
@@
 	1    0    0    -1
 $EndComp
+$Comp
+L LM555N U?
+U 1 1 51CF2CBF
+P 2800 2600
+F 0 "U?" H 2800 2700 70  0000 C CNN
+F 1 "LM555N" H 2800 2500 70  0000 C CNN
+F 2 "" H 2800 2600 60  0000 C CNN
+F 3 "" H 2800 2600 60  0000 C CNN
+	1    2800 2600
+	1    0    0    -1
+$EndComp
+$Comp
+L LM555N U?
+U 1 1 51CF2CD6
+P 2800 3450
+F 0 "U?" H 2800 3550 70  0000 C CNN
+F 1 "LM555N" H 2800 3350 70  0000 C CNN
+F 2 "" H 2800 3450 60  0000 C CNN
+F 3 "" H 2800 3450 60  0000 C CNN
+	1    2800 3450
+	1    0    0    -1
+$EndComp
+Wire Wire Line
+	4100 3450 3500 3450
+Wire Wire Line
+	4100 3650 3500 3650
+Connection ~ 4100 3650
+Wire Wire Line
+	4100 3450 4100 3650
+Wire Wire Line
+	4100 3650 4100 4000
+Wire Wire Line
+	3700 4400 3700 4400
 $EndSCHEMATC

Commit message: 
Parts:
- added D1: LED, ~, symbol LED
- added R4: 680, ~, symbol R
- added SW1: SPST, ~, symbol SPST
- R3: value 4K7 -> 6K8
- RV1, RV2: value 470K -> 500K
- gave numbers to parts that had none: 2
- renumbered C3 to C1, C1 to C3, C2 to C4
Connections:
- net +9V: now also D1.1 (A), SW1.2; no longer BT1.1 (+)
- net GND: now also R4.1
- new net: BT1.1 (+), SW1.1
- new net: D1.2 (K), R4.2
Other:
- moved on the sheet: BT1
Changed lines of the file:
@@
 Sheet 1 1
 Title ""
-Date "29 jun 2013"
+Date "9 jul 2013"
 Rev ""
 Comp ""
@@
 P 4500 3750
 F 0 "RV2" H 4500 3650 50  0000 C CNN
-F 1 "470K" H 4500 3750 50  0000 C CNN
+F 1 "500K" H 4500 3750 50  0000 C CNN
 F 2 "~" H 4500 3750 60  0000 C CNN
 F 3 "~" H 4500 3750 60  0000 C CNN
@@
 P 4200 2350
 F 0 "RV1" H 4200 2250 50  0000 C CNN
-F 1 "470K" H 4200 2350 50  0000 C CNN
+F 1 "500K" H 4200 2350 50  0000 C CNN
 F 2 "~" H 4200 2350 60  0000 C CNN
 F 3 "~" H 4200 2350 60  0000 C CNN
@@
 	3700 2800 3500 2800
 Wire Wire Line
-	3700 1900 3700 2800
-Wire Wire Line
-	3700 2800 3700 4000
+	3700 1900 3700 4000
 Wire Wire Line
 	3700 1900 2100 1900
@@
 Connection ~ 3700 2800
 $Comp
-L C C1
+L C C3
 U 1 1 51CDC33B
 P 3700 4200
-F 0 "C1" H 3700 4300 40  0000 L CNN
+F 0 "C3" H 3700 4300 40  0000 L CNN
 F 1 "10n" H 3706 4115 40  0000 L CNN
 F 2 "~" H 3738 4050 30  0000 C CNN
@@
 $EndComp
 $Comp
-L CP1 C3
+L CP1 C1
 U 1 1 51CDC41A
 P 5100 3250
-F 0 "C3" H 5150 3350 50  0000 L CNN
+F 0 "C1" H 5150 3350 50  0000 L CNN
 F 1 "10u" H 5150 3150 50  0000 L CNN
 F 2 "~" H 5100 3250 60  0000 C CNN
@@
 P 5800 3500
 F 0 "R3" V 5880 3500 40  0000 C CNN
-F 1 "4K7" V 5807 3501 40  0000 C CNN
+F 1 "6K8" V 5807 3501 40  0000 C CNN
 F 2 "~" V 5730 3500 30  0000 C CNN
 F 3 "~" H 5800 3500 30  0000 C CNN
@@
 	4100 4000 4500 4000
 $Comp
-L C C2
+L C C4
 U 1 1 51CDC505
 P 4500 4200
-F 0 "C2" H 4500 4300 40  0000 L CNN
+F 0 "C4" H 4500 4300 40  0000 L CNN
 F 1 "100n" H 4506 4115 40  0000 L CNN
 F 2 "~" H 4538 4050 30  0000 C CNN
@@
 $EndComp
 Wire Wire Line
-	4500 4400 3700 4400
+	3700 4400 4500 4400
 $Comp
 L +9V #PWR05
@@
 	5950 3750 5800 3750
 Wire Wire Line
-	5950 3000 5950 3100
-Wire Wire Line
-	5950 3100 5950 3750
+	5950 3000 5950 3750
 Wire Wire Line
 	5950 3000 6100 3000
@@
 L BATTERY BT1
 U 1 1 51CDC812
-P 5150 2100
-F 0 "BT1" H 5150 2300 50  0000 C CNN
-F 1 "BATTERY" H 5150 1910 50  0000 C CNN
-F 2 "~" H 5150 2100 60  0000 C CNN
-F 3 "~" H 5150 2100 60  0000 C CNN
-	1    5150 2100
+P 5150 2400
+F 0 "BT1" H 5150 2600 50  0000 C CNN
+F 1 "BATTERY" H 5150 2210 50  0000 C CNN
+F 2 "~" H 5150 2400 60  0000 C CNN
+F 3 "~" H 5150 2400 60  0000 C CNN
+	1    5150 2400
 	0    1    1    0
 $EndComp
@@
 L GND #PWR07
 U 1 1 51CDC81F
-P 5150 2400
-F 0 "#PWR07" H 5150 2400 30  0001 C CNN
-F 1 "GND" H 5150 2330 30  0001 C CNN
-F 2 "" H 5150 2400 60  0000 C CNN
-F 3 "" H 5150 2400 60  0000 C CNN
-	1    5150 2400
+P 5150 2700
+F 0 "#PWR07" H 5150 2700 30  0001 C CNN
+F 1 "GND" H 5150 2630 30  0001 C CNN
+F 2 "" H 5150 2700 60  0000 C CNN
+F 3 "" H 5150 2700 60  0000 C CNN
+	1    5150 2700
 	1    0    0    -1
 $EndComp
@@
 L +9V #PWR08
 U 1 1 51CDC825
-P 5150 1800
-F 0 "#PWR08" H 5150 1770 20  0001 C CNN
-F 1 "+9V" H 5150 1910 30  0000 C CNN
-F 2 "" H 5150 1800 60  0000 C CNN
-F 3 "" H 5150 1800 60  0000 C CNN
-	1    5150 1800
-	1    0    0    -1
-$EndComp
-$Comp
-L LM555N U?
+P 6150 1850
+F 0 "#PWR08" H 6150 1820 20  0001 C CNN
+F 1 "+9V" H 6150 1960 30  0000 C CNN
+F 2 "" H 6150 1850 60  0000 C CNN
+F 3 "" H 6150 1850 60  0000 C CNN
+	1    6150 1850
+	1    0    0    -1
+$EndComp
+$Comp
+L LM555N U1
 U 1 1 51CF2CBF
 P 2800 2600
-F 0 "U?" H 2800 2700 70  0000 C CNN
+F 0 "U1" H 2800 2700 70  0000 C CNN
 F 1 "LM555N" H 2800 2500 70  0000 C CNN
 F 2 "" H 2800 2600 60  0000 C CNN
@@
 $EndComp
 $Comp
-L LM555N U?
+L LM555N U2
 U 1 1 51CF2CD6
 P 2800 3450
-F 0 "U?" H 2800 3550 70  0000 C CNN
+F 0 "U2" H 2800 3550 70  0000 C CNN
 F 1 "LM555N" H 2800 3350 70  0000 C CNN
 F 2 "" H 2800 3450 60  0000 C CNN
@@
 Connection ~ 4100 3650
 Wire Wire Line
-	4100 3450 4100 3650
-Wire Wire Line
-	4100 3650 4100 4000
-Wire Wire Line
-	3700 4400 3700 4400
+	4100 3450 4100 4000
+$Comp
+L LED D1
+U 1 1 51DC96FD
+P 6350 2100
+F 0 "D1" H 6350 2200 50  0000 C CNN
+F 1 "LED" H 6350 2000 50  0000 C CNN
+F 2 "~" H 6350 2100 60  0000 C CNN
+F 3 "~" H 6350 2100 60  0000 C CNN
+	1    6350 2100
+	1    0    0    -1
+$EndComp
+$Comp
+L R R4
+U 1 1 51DC970A
+P 6800 2100
+F 0 "R4" V 6880 2100 40  0000 C CNN
+F 1 "680" V 6807 2101 40  0000 C CNN
+F 2 "~" V 6730 2100 30  0000 C CNN
+F 3 "~" H 6800 2100 30  0000 C CNN
+	1    6800 2100
+	0    1    1    0
+$EndComp
+$Comp
+L GND #PWR09
+U 1 1 51DC9710
+P 7050 2200
+F 0 "#PWR09" H 7050 2200 30  0001 C CNN
+F 1 "GND" H 7050 2130 30  0001 C CNN
+F 2 "" H 7050 2200 60  0000 C CNN
+F 3 "" H 7050 2200 60  0000 C CNN
+	1    7050 2200
+	1    0    0    -1
+$EndComp
+Wire Wire Line
+	7050 2100 7050 2200
+$Comp
+L SPST SW1
+U 1 1 51DC98CA
+P 5650 2100
+F 0 "SW1" H 5650 2200 70  0000 C CNN
+F 1 "SPST" H 5650 2000 70  0000 C CNN
+F 2 "~" H 5650 2100 60  0000 C CNN
+F 3 "~" H 5650 2100 60  0000 C CNN
+	1    5650 2100
+	1    0    0    -1
+$EndComp
+Wire Wire Line
+	6150 1850 6150 2100
 $EndSCHEMATC

Commit message: 
Parts:
- removed D1: LED, ~, symbol LED
- removed R4: 680, ~, symbol R
- removed SW1: SPST, ~, symbol SPST
Connections:
- net +9V: now also BT1.1 (+)
Changed lines of the file:
@@
 Sheet 1 1
 Title ""
-Date "9 jul 2013"
+Date "8 sep 2013"
 Rev ""
 Comp ""
@@
 L +9V #PWR08
 U 1 1 51CDC825
-P 6150 1850
-F 0 "#PWR08" H 6150 1820 20  0001 C CNN
-F 1 "+9V" H 6150 1960 30  0000 C CNN
-F 2 "" H 6150 1850 60  0000 C CNN
-F 3 "" H 6150 1850 60  0000 C CNN
-	1    6150 1850
+P 5150 2050
+F 0 "#PWR08" H 5150 2020 20  0001 C CNN
+F 1 "+9V" H 5150 2160 30  0000 C CNN
+F 2 "" H 5150 2050 60  0000 C CNN
+F 3 "" H 5150 2050 60  0000 C CNN
+	1    5150 2050
 	1    0    0    -1
 $EndComp
@@
 Wire Wire Line
 	4100 3450 4100 4000
-$Comp
-L LED D1
-U 1 1 51DC96FD
-P 6350 2100
-F 0 "D1" H 6350 2200 50  0000 C CNN
-F 1 "LED" H 6350 2000 50  0000 C CNN
-F 2 "~" H 6350 2100 60  0000 C CNN
-F 3 "~" H 6350 2100 60  0000 C CNN
-	1    6350 2100
-	1    0    0    -1
-$EndComp
-$Comp
-L R R4
-U 1 1 51DC970A
-P 6800 2100
-F 0 "R4" V 6880 2100 40  0000 C CNN
-F 1 "680" V 6807 2101 40  0000 C CNN
-F 2 "~" V 6730 2100 30  0000 C CNN
-F 3 "~" H 6800 2100 30  0000 C CNN
-	1    6800 2100
-	0    1    1    0
-$EndComp
-$Comp
-L GND #PWR09
-U 1 1 51DC9710
-P 7050 2200
-F 0 "#PWR09" H 7050 2200 30  0001 C CNN
-F 1 "GND" H 7050 2130 30  0001 C CNN
-F 2 "" H 7050 2200 60  0000 C CNN
-F 3 "" H 7050 2200 60  0000 C CNN
-	1    7050 2200
-	1    0    0    -1
-$EndComp
-Wire Wire Line
-	7050 2100 7050 2200
-$Comp
-L SPST SW1
-U 1 1 51DC98CA
-P 5650 2100
-F 0 "SW1" H 5650 2200 70  0000 C CNN
-F 1 "SPST" H 5650 2000 70  0000 C CNN
-F 2 "~" H 5650 2100 60  0000 C CNN
-F 3 "~" H 5650 2100 60  0000 C CNN
-	1    5650 2100
-	1    0    0    -1
-$EndComp
-Wire Wire Line
-	6150 1850 6150 2100
+Wire Wire Line
+	5150 2050 5150 2100
 $EndSCHEMATC
